File: hardware/robot_chat/robot_chat.kicad_pcb (KiCad board)
At the start: 2 copper layers, 90 x 72 mm, 55 parts, among them J102 BATTERY, J103 BORDER_FRONT, J104 BORDER_BACK, J105 BUMPER, J106 M1, J107 M2, J108 LIDAR, J7 Conn_02x07_Odd_Even, SW101 SW_SPDT, U101 STM32G070RBT6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

Commit message: place + started routing
Parts:
- added D103: GREEN, LED_SMD:LED_0603_1608Metric, F.Cu at (143.2, 87.0)
- added D104: ORANGE, LED_SMD:LED_0603_1608Metric, F.Cu at (143.2, 89.6)
- added D105: RED, LED_SMD:LED_0603_1608Metric, F.Cu at (143.2, 92.2)
- added J109: BUMPER2, Connector_JST:JST_XH_S2B-XH-A_1x02_P2.50mm_Horizontal, F.Cu at (110.2, 35.5)
- added J110: BUMPER1, Connector_JST:JST_XH_S2B-XH-A_1x02_P2.50mm_Horizontal, F.Cu at (101.2, 35.5)
- added J111: BUMPER3, Connector_JST:JST_XH_S2B-XH-A_1x02_P2.50mm_Horizontal, F.Cu at (119.2, 35.5)
- added R109: 1k, Resistor_SMD:R_0603_1608Metric, F.Cu at (147.2, 87.0)
- added R110: 1k, Resistor_SMD:R_0603_1608Metric, F.Cu at (147.2, 89.5)
- added R111: 1k, Resistor_SMD:R_0603_1608Metric, F.Cu at (147.2, 92.0)
- J105: value BUMPER -> BUMPER0
- moved U102 56.4 mm to (85.5, 53.0), turned to 90 degrees
- moved R107 52.7 mm to (81.2, 51.0), turned to -90 degrees
- moved R108 52.2 mm to (82.9, 47.9), turned to 90 degrees
- moved R104 51.4 mm to (82.1, 56.7), turned to 180 degrees
- moved R106 50.7 mm to (82.9, 51.0), turned to -90 degrees
- moved R103 49.4 mm to (82.1, 54.1)
- moved D102 47.1 mm to (85.8, 47.9), turned to 180 degrees
- moved U103 47.1 mm to (96.1, 59.0), turned to 90 degrees
- moved C116 46.1 mm to (81.2, 47.9), turned to -90 degrees
- moved R105 45.1 mm to (88.4, 48.8), turned to 90 degrees
- moved J102 41.8 mm to (85.5, 83.5)
- moved C114 40.3 mm to (85.5, 50.0)
- moved C113 39.5 mm to (85.8, 56.7)
- moved L101 38.3 mm to (91.5, 53.0), turned to -90 degrees
- moved R102 37.1 mm to (96.5, 49.1), turned to 90 degrees
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Connections:
- net Net-(C116-Pad2) renamed /BUCK_FB_MID
- net Net-(D102-K) renamed /BUCK_BST_MID
- net Net-(U102-BST) renamed /BUCK_BST
- net Net-(U102-EN/SYNC) renamed /BUCK_EN
- net Net-(U102-FB) renamed /BUCK_FB
- net Net-(U102-PG) renamed /BUCK_PG
- net Net-(U102-SW) renamed /BUCK_SW
- C110 pad 1: Net-(U102-IN) -> +BATT
- C113 pad 1: Net-(U102-IN) -> +BATT
- J103 pad 1: unconnected-(J103-Pin_1-Pad1) -> GND
- J103 pad 2: unconnected-(J103-Pin_2-Pad2) -> +3.3V
- J103 pad 3: unconnected-(J103-Pin_3-Pad3) -> /BORDER_FRONT
- J104 pad 1: unconnected-(J104-Pin_1-Pad1) -> GND
- J104 pad 2: unconnected-(J104-Pin_2-Pad2) -> +3.3V
- J104 pad 3: unconnected-(J104-Pin_3-Pad3) -> /BORDER_BACK
- J105 pad 1: unconnected-(J105-Pin_1-Pad1) -> /BUMPER0
- J105 pad 2: unconnected-(J105-Pin_2-Pad2) -> GND
- J106 pad 1: unconnected-(J106-Pin_1-Pad1) -> /M1_OUT2
- J106 pad 2: unconnected-(J106-Pin_2-Pad2) -> GND
- J106 pad 3: unconnected-(J106-Pin_3-Pad3) -> /M1_QEI_A
- J106 pad 4: unconnected-(J106-Pin_4-Pad4) -> /M1_QEI_B
- J106 pad 5: unconnected-(J106-Pin_5-Pad5) -> +3.3V
- J106 pad 6: unconnected-(J106-Pin_6-Pad6) -> /M1_OUT1
- J107 pad 1: unconnected-(J107-Pin_1-Pad1) -> /M2_OUT2
- J107 pad 2: unconnected-(J107-Pin_2-Pad2) -> GND
- J107 pad 3: unconnected-(J107-Pin_3-Pad3) -> /M2_QEI_A
- J107 pad 4: unconnected-(J107-Pin_4-Pad4) -> /M2_QEI_B
- J107 pad 5: unconnected-(J107-Pin_5-Pad5) -> +3.3V
- J107 pad 6: unconnected-(J107-Pin_6-Pad6) -> /M2_OUT1
- R104 pad 1: Net-(U102-IN) -> +BATT
- U101 pad 19: /M1_PWM_FWD -> unconnected-(U101-PA2-Pad19)
- U101 pad 2: /LIDAR_PWM -> unconnected-(U101-PC12-Pad2)
- U101 pad 20: /M1_PWM_REV -> unconnected-(U101-PA3-Pad20)
- U101 pad 23: /M2_PWM_FWD -> unconnected-(U101-PA6-Pad23)
- U101 pad 24: /M2_PWM_REV -> unconnected-(U101-PA7-Pad24)
- U101 pad 28: unconnected-(U101-PB1-Pad28) -> /LIDAR_M_SCTR
- U101 pad 34: unconnected-(U101-PB14-Pad34) -> /M2_PWM_REV
- U101 pad 35: unconnected-(U101-PB15-Pad35) -> /M2_PWM_FWD
- U101 pad 36: /M1_QEI_B -> /M2_QEI_B
- U101 pad 37: /M1_QEI_A -> /M2_QEI_A
- U101 pad 38: /M2_QEI_B -> /M1_QEI_B
- U101 pad 39: /M2_QEI_A -> /M1_QEI_A
- U101 pad 50: unconnected-(U101-PD0-Pad50) -> /M1_PWM_REV
- U101 pad 51: unconnected-(U101-PD1-Pad51) -> /M1_PWM_FWD
- U102 pad 2: Net-(U102-IN) -> +BATT
- U102 pad 4: (no net) -> GND
Routing:
- net /M1_QEI_B: track 0.00 -> 51.3 mm
- net /M2_QEI_A: track 0.00 -> 48.1 mm
- net /M1_QEI_A: track 0.00 -> 48.1 mm
- net /M2_QEI_B: track 0.00 -> 44.3 mm
- net GND: track 0.00 -> 33.8 mm, vias 0 -> 27
- net /M1_PWM_REV: track 0.00 -> 33.6 mm
- net /M1_PWM_FWD: track 0.00 -> 32.4 mm
- net +BATT: track 0.00 -> 30.9 mm
- net /M2_PWM_REV: track 0.00 -> 27.7 mm
- net +5V: track 0.00 -> 25.4 mm, vias 0 -> 2
- net /M2_PWM_FWD: track 0.00 -> 23.2 mm
- net /LIDAR_M_SCTR: track 0.00 -> 22.7 mm
- net +3.3V: track 0.00 -> 13.6 mm
- net /BUCK_VCC: track 0.00 -> 12.9 mm, vias 0 -> 2
- net /BUCK_EN: track 0.00 -> 11.0 mm, vias 0 -> 2
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- added copper zone on F.Cu, net +5V
- added copper zone on F.Cu, net +BATT
- added copper zone on B.Cu, net /BUCK_SW
- added copper zone on F.Cu, net /BUCK_SW
- added copper zone on B.Cu, net GND

Commit message: routage
Parts:
- moved D103 22.6 mm to (131.0, 68.0), turned to 180 degrees
- moved R109 22.5 mm to (135.0, 68.0)
- moved D104 22.2 mm to (131.0, 71.0), turned to 180 degrees
- moved R110 22.1 mm to (135.0, 71.0)
- moved D105 21.9 mm to (131.0, 74.0), turned to 180 degrees
- moved R111 21.7 mm to (135.0, 74.0)
Connections:
- U101 pad 17: unconnected-(U101-PA0-Pad17) -> /LIDAR_TX
- U101 pad 18: unconnected-(U101-PA1-Pad18) -> /LIDAR_RX
- U101 pad 55: unconnected-(U101-PD5-Pad55) -> /STLINK_RX
- U101 pad 56: unconnected-(U101-PD6-Pad56) -> /STLINK_TX
- U101 pad 60: unconnected-(U101-PB6-Pad60) -> /BUMPER3
- U101 pad 61: unconnected-(U101-PB7-Pad61) -> /BUMPER2
- U101 pad 62: unconnected-(U101-PB8-Pad62) -> /BUMPER1
- U101 pad 63: unconnected-(U101-PB9-Pad63) -> /BUMPER0
Routing:
- net /BORDER_BACK: track 0.00 -> 34.8 mm
- net /BUMPER2: track 0.00 -> 27.1 mm
- net /LIDAR_TX: track 0.00 -> 21.9 mm
- net /NRST: track 3.32 -> 25.1 mm
- net /LIDAR_RX: track 0.00 -> 21.1 mm
- net /BUMPER3: track 0.00 -> 20.9 mm
- net /BORDER_FRONT: track 0.00 -> 20.6 mm
- net /STLINK_RX: track 0.00 -> 18.3 mm
- net /STLINK_TX: track 0.00 -> 13.4 mm
- net Net-(D105-K): track 0.00 -> 2.39 mm
- net Net-(D104-K): track 0.00 -> 2.39 mm
- net Net-(D103-K): track 0.00 -> 2.39 mm
- net GND: track 33.8 -> 35.8 mm, vias 27 -> 30

Commit message: routing
Parts:
- added G***: LOGO, logo_ensea:logo_ensea_15mm, F.Cu at (142.0, 87.0)
- added TP101: M1_PWM_FWD, TestPoint:TestPoint_Pad_D1.5mm, F.Cu at (143.7, 46.5)
- added TP102: M1_PWM_REV, TestPoint:TestPoint_Pad_D1.5mm, F.Cu at (143.7, 49.4)
- added TP103: M2_PWM_FWD, TestPoint:TestPoint_Pad_D1.5mm, F.Cu at (143.7, 69.1)
- added TP104: M2_PWM_REV, TestPoint:TestPoint_Pad_D1.5mm, F.Cu at (143.7, 72.0)
- moved C121 13.1 mm to (152.7, 56.4), turned to -90 degrees
- moved C122 12.3 mm to (152.0, 43.0), turned to 90 degrees
- moved C123 0.73 mm to (152.7, 81.2)
- moved J103 0.50 mm to (137.0, 35.5)
- moved C117 0.30 mm to (148.0, 43.0)
- moved C6 0.30 mm to (150.0, 43.0)
Connections:
- net Net-(J102-Pin_1) renamed /BATT_OUT
- J7 pad 8: /SWO -> unconnected-(J101-Pin_8-Pad8)
- U101 pad 25: unconnected-(U101-PC4-Pad25) -> /LIDAR_M_EN
- U101 pad 26: unconnected-(U101-PC5-Pad26) -> /LIDAR_DEV_EN
- U101 pad 31: unconnected-(U101-PB11-Pad31) -> /LED_RED
- U101 pad 32: unconnected-(U101-PB12-Pad32) -> /LED_ORANGE
- U101 pad 33: unconnected-(U101-PB13-Pad33) -> /LED_GREEN
- U101 pad 52: unconnected-(U101-PD2-Pad52) -> /BORDER_BACK
- U101 pad 53: unconnected-(U101-PD3-Pad53) -> /BORDER_FRONT
Routing:
- net +3.3V: track 13.6 -> 139.4 mm, vias 0 -> 2
- net /BUMPER0: track 0.00 -> 43.7 mm
- net +5V: track 25.4 -> 67.4 mm, vias 2 -> 6
- net /BUMPER1: track 0.00 -> 35.4 mm
- net /LIDAR_DEV_EN: track 0.00 -> 22.1 mm
- net /LIDAR_M_EN: track 0.00 -> 21.3 mm
- net GND: track 35.8 -> 53.8 mm, vias 30 -> 78
- net /LED_RED: track 0.00 -> 11.3 mm
- net +BATT: track 30.9 -> 40.7 mm, vias 0 -> 28
- net /LED_ORANGE: track 0.00 -> 8.00 mm
- net /BORDER_FRONT: track 20.6 -> 27.3 mm
- net /LED_GREEN: track 0.00 -> 5.17 mm
- net /BORDER_BACK: track 34.8 -> 37.4 mm
- net /M2_PWM_REV: track 27.7 -> 26.5 mm
- added copper zone on B.Cu, net +BATT
- added copper zone on F.Cu, net /BATT_OUT
- added copper zone on F.Cu, net /M1_OUT1
- added copper zone on F.Cu, net /M1_OUT2
- added copper zone on F.Cu, net /M2_OUT1
- added copper zone on F.Cu, net /M2_OUT2
- added copper zone on F.Cu, net GND
Other:
- board text added: "( o.o )"
- board text added: "+"
- board text added: "-"
- board text added: "/\_/\"
- board text added: "> ^ <"
- board text added: "BACK"
- board text added: "BATTERY"
- board text added: "BUMPER0"
- board text added: "BUMPER1"
- board text added: "BUMPER2"
- board text added: "BUMPER3"
- board text added: "FRONT"
- board text added: "FWD"
- board text added: "JLCJLCJLCJLC"
- board text added: "LIDAR"
- board text added: "MOTOR1"
- board text added: "MOTOR2"
- board text added: "RED"
- board text added: "REV"
- board text added: "ROBOT CHAT"
- board text added: "v0.0 - 2023/10 Laurent Fiack"
