File: hardware/robot_chat/robot_chat.kicad_sch (KiCad schematic)
At the start: 2 parts, among them U101 STM32G070RBTx, U102 MP1475

Commit message: schematic
Parts:
- added C101, C102: 10pF, Capacitor_SMD:C_0603_1608Metric, symbol Device:C_Small
- added C103: 4.7uF, Capacitor_SMD:C_0603_1608Metric, symbol Device:C_Small
- added C104, C105, C106, C107, C113, C114, C115, C121, C122, C123, C124: 100nF, Capacitor_SMD:C_0603_1608Metric, symbol Device:C_Small
- added C108, C109, C117, C120: 1uF, Capacitor_SMD:C_0603_1608Metric, symbol Device:C_Small
- added C110, C111, C112: 22uF, Capacitor_SMD:C_0805_2012Metric, symbol Device:C_Small
- added C116: 15pF, Capacitor_SMD:C_0603_1608Metric, symbol Device:C_Small
- added C125: 220uF, Capacitor_SMD:CP_Elec_8x10.5, symbol Device:C_Polarized_Small
- added C6 (x2): 10uF, Capacitor_SMD:C_0603_1608Metric_Pad1.08x0.95mm_HandSolder, symbol Device:C_Small
- added D101: BLUE, LED_SMD:LED_0603_1608Metric, symbol Device:LED_Small
- added D102: D_Small, Diode_SMD:D_SOD-323, symbol Device:D_Small
- added H101, H102, H103, H104: MountingHole_Pad, MountingHole:MountingHole_3.2mm_M3_Pad_Via, symbol Mechanical:MountingHole_Pad
- added J102: BATTERY, Connector_JST:JST_XH_S2B-XH-A_1x02_P2.50mm_Horizontal, symbol Connector_Generic:Conn_01x02
- added J103: BORDER_FRONT, Connector_JST:JST_XH_S3B-XH-A_1x03_P2.50mm_Horizontal, symbol Connector_Generic:Conn_01x03
- added J104: BORDER_BACK, Connector_JST:JST_XH_S3B-XH-A_1x03_P2.50mm_Horizontal, symbol Connector_Generic:Conn_01x03
- added J105: BUMPER, Connector_JST:JST_XH_S2B-XH-A_1x02_P2.50mm_Horizontal, symbol Connector_Generic:Conn_01x02
- added J106: M1, Connector_JST:JST_XH_S6B-XH-A_1x06_P2.50mm_Horizontal, symbol Connector_Generic:Conn_01x06
- added J107: M2, Connector_JST:JST_XH_S6B-XH-A_1x06_P2.50mm_Horizontal, symbol Connector_Generic:Conn_01x06
- added J108: LIDAR, Connector_JST:JST_XH_S8B-XH-A_1x08_P2.50mm_Horizontal, symbol Connector_Generic:Conn_01x08
- added J7: Conn_02x07_Odd_Even, Connector_PinHeader_1.27mm:PinHeader_2x07_P1.27mm_Vertical_SMD, symbol Connector_Generic:Conn_02x07_Odd_Even
- added L101: 4.7uH, Inductor_SMD:L_1008_2520Metric, symbol Device:L_Small
- added R101: 10R, Resistor_SMD:R_0603_1608Metric, symbol Device:R_Small
- added R102: 1k, Resistor_SMD:R_0603_1608Metric, symbol Device:R_Small
- added R103, R104: 100k, Resistor_SMD:R_0603_1608Metric, symbol Device:R_Small
- added R105: 20R, Resistor_SMD:R_0603_1608Metric, symbol Device:R_Small
- added R106: 16k, Resistor_SMD:R_0603_1608Metric, symbol Device:R_Small
- added R107: 7.68k, Resistor_SMD:R_0603_1608Metric, symbol Device:R_Small
- added R108: 40.2k, Resistor_SMD:R_0603_1608Metric, symbol Device:R_Small
- added SW101: SW_SPDT, 472121020421:Toggle_Switch, symbol Switch:SW_SPDT
- added U103: BU33SD5WG-TR, Package_TO_SOT_SMD:SOT-23-5, symbol WITNS_ROHM:BU33SD5WG-TR
- added U104, U105: ZXBM5210-SP, Package_SO:Diodes_SO-8EP, symbol Driver_Motor:ZXBM5210-SP
- added Y101: 16MHz, Crystal:Crystal_SMD_EuroQuartz_MT-4Pin_3.2x2.5mm, symbol Device:Crystal_GND24_Small
- U101: value STM32G070RBTx -> STM32G070RBT6
- U102: value MP1475 -> MP1475DJ-LF-P
Connections:
- net GND: now reaches U102. (GND)
- net GND: now also U101.9 (VSS), C101.1, C102.1, C103.2, C104.2, C105.2, C106.2, C107.1, C108.2, C109.2, C110.2, C111.2, C112.2, C113.2, C114.2, C117.2, C120.2, C121.2, C122.2, C123.2, C124.2, C125.2, C6.2, C6.2, H101.1, H102.1, H103.1, H104.1, J102.2 (Pin_2), J108.4 (Pin_4), J7.11 (Pin_11), J7.5 (Pin_5), J7.7 (Pin_7), R102.2, R107.2, U103.2 (GND), U104.8 (GND), U104.9 (GND), U105.8 (GND), U105.9 (GND), Y101.2, Y101.4
- net at U102.1 (PG): now also R103.2
- net at U102.2 (IN): now also C110.1, C113.1, R104.1
- net at U102.3 (SW): now also C115.2, L101.1
- net at U102.5 (BST): now also R105.1
- net at U102.6 (EN/SYNC): now also R104.2
- net BUCK_VCC: now reaches U102.7 (VCC)
- net BUCK_VCC: now also C114.1, D102.2 (A), R103.1
- net at U102.8 (FB): now also R106.2
- net OSC_IN: now reaches U101.10 (PF0)
- net OSC_IN: now also C101.2, Y101.3
- net OSC_OUT: now reaches U101.11 (PF1)
- net OSC_OUT: now also R101.2
- net NRST: now reaches U101.12 (NRST)
- net NRST: now also C107.2, J7.12 (Pin_12)
- net M1_PWM_FWD: now reaches U101.19 (PA2)
- net M1_PWM_FWD: now also U104.4 (FWD)
- net LIDAR_PWM: now reaches U101.2 (PC12)
- net M1_PWM_REV: now reaches U101.20 (PA3)
- net M1_PWM_REV: now also U104.5 (REV)
- net M2_PWM_FWD: now reaches U101.23 (PA6)
- net M2_PWM_FWD: now also U105.4 (FWD)
- net M2_PWM_REV: now reaches U101.24 (PA7)
- net M2_PWM_REV: now also U105.5 (REV)
- net M1_QEI_B: now reaches U101.36 (PA8)
- net M1_QEI_A: now reaches U101.37 (PA9/NC)
- net M2_QEI_B: now reaches U101.38 (PC6)
- net M2_QEI_A: now reaches U101.39 (PC7)
- net SWDIO: now reaches U101.45 (PA13)
- net SWDIO: now also J7.4 (Pin_4)
- net SWCLK: now reaches U101.46 (PA14)
- net SWCLK: now also J7.6 (Pin_6)
- net +3.3V: now reaches U101.6 (VBAT)
- net +3.3V: now also U101.7 (VREF+), U101.8 (VDD), C103.1, C104.1, C105.1, C106.1, C108.1, D101.2 (A), J7.3 (Pin_3), U103.5 (OUT)
- new net: C116.2, R106.1, R107.1, R108.1
- new net: C115.1, D102.1 (K), R105.2
- new net: J102.1 (Pin_1), SW101.1 (A)
- new net: D101.1 (K), R102.1
- new net +5V: C109.1, C111.1, C112.1, C116.1, J108.1 (Pin_1), L101.2, R108.2, U103.1 (IN), U103.3 (STBY)
- new net +BATT: C117.1, C120.1, C125.1, C6.1, C6.1, SW101.2 (B), U104.2 (VM), U104.3 (VDD), U104.6 (VREF), U105.2 (VM), U105.3 (VDD), U105.6 (VREF)
- new net LIDAR_DEV_EN: J108.6 (Pin_6)
- new net LIDAR_M_EN: J108.5 (Pin_5)
- new net LIDAR_M_SCTR: J108.7 (Pin_7)
- new net LIDAR_RX: J108.3 (Pin_3)
- new net LIDAR_TX: J108.2 (Pin_2)
- new net M1_OUT1: C122.1, U104.1 (OUT1)
- new net M1_OUT2: C121.1, U104.7 (OUT2)
- new net M2_OUT1: C124.1, U105.1 (OUT1)
- new net M2_OUT2: C123.1, U105.7 (OUT2)
- new net STLINK_RX: J7.13 (Pin_13)
- new net STLINK_TX: J7.14 (Pin_14)
- new net SWO: J7.8 (Pin_8)
- new net XTAL1: C102.2, R101.1, Y101.1
- no-connect marks 0 -> 6
Other:
- note added: "Bypass capacitors 100nF as close to STM32 VDD as possible 4.7uF just next to the 100nF"
- note added: "TODO Replace?"
- moved on the sheet: U101, U102

Commit message: place + started routing
Parts:
- added D103: GREEN, LED_SMD:LED_0603_1608Metric, symbol Device:LED_Small
- added D104: ORANGE, LED_SMD:LED_0603_1608Metric, symbol Device:LED_Small
- added D105: RED, LED_SMD:LED_0603_1608Metric, symbol Device:LED_Small
- added J109: BUMPER2, Connector_JST:JST_XH_S2B-XH-A_1x02_P2.50mm_Horizontal, symbol Connector_Generic:Conn_01x02
- added J110: BUMPER1, Connector_JST:JST_XH_S2B-XH-A_1x02_P2.50mm_Horizontal, symbol Connector_Generic:Conn_01x02
- added J111: BUMPER3, Connector_JST:JST_XH_S2B-XH-A_1x02_P2.50mm_Horizontal, symbol Connector_Generic:Conn_01x02
- added R109, R110, R111: 1k, Resistor_SMD:R_0603_1608Metric, symbol Device:R_Small
- J105: value BUMPER -> BUMPER0
Connections:
- net +3.3V: now also J103.2 (Pin_2), J104.2 (Pin_2), J106.5 (Pin_5), J107.5 (Pin_5)
- net +BATT: now also C110.1, C113.1, R104.1, U102.2 (IN)
- net GND: now also J103.1 (Pin_1), J104.1 (Pin_1), J105.2 (Pin_2), J106.2 (Pin_2), J107.2 (Pin_2), U102.4 (GND), J109.2 (Pin_2), J110.2 (Pin_2), J111.2 (Pin_2), R109.2, R110.2, R111.2; no longer U102. (GND)
- net LIDAR_M_SCTR: now also U101.28 (PB1)
- net M1_OUT1: now also J106.6 (Pin_6)
- net M1_OUT2: now also J106.1 (Pin_1)
- net M1_PWM_FWD: now also U101.51 (PD1); no longer U101.19 (PA2)
- net M1_PWM_REV: now also U101.50 (PD0); no longer U101.20 (PA3)
- net M1_QEI_A: now also J106.3 (Pin_3), U101.39 (PC7); no longer U101.37 (PA9/NC)
- net M1_QEI_B: now also J106.4 (Pin_4), U101.38 (PC6); no longer U101.36 (PA8)
- net M2_OUT1: now also J107.6 (Pin_6)
- net M2_OUT2: now also J107.1 (Pin_1)
- net M2_PWM_FWD: now also U101.35 (PB15); no longer U101.23 (PA6)
- net M2_PWM_REV: now also U101.34 (PB14); no longer U101.24 (PA7)
- net M2_QEI_A: now also J107.3 (Pin_3), U101.37 (PA9/NC); no longer U101.39 (PC7)
- net M2_QEI_B: now also J107.4 (Pin_4), U101.36 (PA8); no longer U101.38 (PC6)
- net BUCK_FB_MID: now reaches C116.2, R106.1, R107.1, R108.1
- net BUCK_FB: now reaches R106.2, U102.8 (FB)
- net BUCK_PG: now reaches R103.2, U102.1 (PG)
- net BUCK_SW: now reaches C115.2, L101.1, U102.3 (SW)
- net BUCK_BST: now reaches R105.1, U102.5 (BST)
- net BUCK_EN: now reaches R104.2, U102.6 (EN/SYNC)
- net BUCK_BST_MID: now reaches C115.1, D102.1 (K), R105.2
- net BUMPER0: now reaches J105.1 (Pin_1)
- net BORDER_BACK: now reaches J104.3 (Pin_3)
- net BORDER_FRONT: now reaches J103.3 (Pin_3)
- net LIDAR_PWM: no longer names the net of U101.2 (PC12)
- new net: D104.1 (K), R110.1
- new net: D103.1 (K), R109.1
- new net: D105.1 (K), R111.1
- new net BUMPER1: J110.1 (Pin_1)
- new net BUMPER2: J109.1 (Pin_1)
- new net BUMPER3: J111.1 (Pin_1)
- new net LED_GREEN: D103.2 (A)
- new net LED_ORANGE: D104.2 (A)
- new net LED_RED: D105.2 (A)
Other:
- note added: "LIDAR_M_SCTR = PWM"
- note removed: "TODO Replace?"
- moved on the sheet: C101, C102, J103, J104, J105, J106, J107, J108, R101, Y101

Commit message: routage
Connections:
- net BUMPER0: now also U101.63 (PB9)
- net BUMPER1: now also U101.62 (PB8)
- net BUMPER2: now also U101.61 (PB7)
- net BUMPER3: now also U101.60 (PB6)
- net LIDAR_RX: now also U101.18 (PA1)
- net LIDAR_TX: now also U101.17 (PA0)
- net STLINK_RX: now also U101.55 (PD5)
- net STLINK_TX: now also U101.56 (PD6)
Changed lines of the file:
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@@
+    (stroke (width 0) (type default))
+  )
+  (wire (pts (xy 184.15 40.64) (xy 194.31 40.64))
     (stroke (width 0) (type default))
   )
@@
     (stroke (width 0) (type default))
   )
+  (wire (pts (xy 184.15 101.6) (xy 194.31 101.6))
+    (stroke (width 0) (type default))
+  )
   (wire (pts (xy 223.52 52.07) (xy 223.52 53.34))
     (stroke (width 0) (type default))
@@
     (stroke (width 0) (type default))
   )
+  (wire (pts (xy 184.15 104.14) (xy 194.31 104.14))
+    (stroke (width 0) (type default))
+  )
   (wire (pts (xy 92.71 144.78) (xy 101.6 144.78))
     (stroke (width 0) (type default))
@@
     (stroke (width 0) (type default))
   )
+  (wire (pts (xy 184.15 43.18) (xy 194.31 43.18))
+    (stroke (width 0) (type default))
+  )
   (wire (pts (xy 223.52 50.8) (xy 223.52 52.07))
     (stroke (width 0) (type default))
@@
     (stroke (width 0) (type default))
   )
+  (wire (pts (xy 184.15 99.06) (xy 194.31 99.06))
+    (stroke (width 0) (type default))
+  )
   (wire (pts (xy 48.26 26.67) (xy 46.99 26.67))
     (stroke (width 0) (type default))
   )
+  (wire (pts (xy 142.24 71.12) (xy 153.67 71.12))
+    (stroke (width 0) (type default))
+  )
   (wire (pts (xy 74.93 132.08) (xy 72.39 132.08))
     (stroke (width 0) (type default))
@@
     (stroke (width 0) (type default))
   )
+  (wire (pts (xy 184.15 106.68) (xy 194.31 106.68))
+    (stroke (width 0) (type default))
+  )
   (wire (pts (xy 116.84 60.96) (xy 120.65 60.96))
     (stroke (width 0) (type default))
@@
   )
   (wire (pts (xy 184.15 121.92) (xy 198.12 121.92))
+    (stroke (width 0) (type default))
+  )
+  (wire (pts (xy 142.24 73.66) (xy 153.67 73.66))
     (stroke (width 0) (type default))
   )
@@
     (effects (font (size 1.27 1.27)) (justify right bottom))
   )
+  (label "STLINK_TX" (at 142.24 73.66 0) (fields_autoplaced)
+    (effects (font (size 1.27 1.27)) (justify left bottom))
+  )
   (label "SWDIO" (at 265.43 29.21 180) (fields_autoplaced)
     (effects (font (size 1.27 1.27)) (justify right bottom))
@@
     (effects (font (size 1.27 1.27)) (justify right bottom))
   )
-  (label "BUMPER1" (at 132.08 83.82 180) (fields_autoplaced)
+  (label "BUMPER1" (at 194.31 104.14 180) (fields_autoplaced)
     (effects (font (size 1.27 1.27)) (justify right bottom))
   )
@@
     (effects (font (size 1.27 1.27)) (justify right bottom))
   )
+  (label "STLINK_RX" (at 142.24 71.12 0) (fields_autoplaced)
+    (effects (font (size 1.27 1.27)) (justify left bottom))
+  )
   (label "M1_PWM_FWD" (at 229.87 63.5 0) (fields_autoplaced)
     (effects (font (size 1.27 1.27)) (justify left bottom))
   )
-  (label "BUMPER0" (at 132.08 81.28 180) (fields_autoplaced)
+  (label "BUMPER0" (at 194.31 106.68 180) (fields_autoplaced)
     (effects (font (size 1.27 1.27)) (justify right bottom))
   )
@@
     (effects (font (size 1.27 1.27)) (justify right bottom))
   )
-  (label "LIDAR_TX" (at 127 99.06 180) (fields_autoplaced)
-    (effects (font (size 1.27 1.27)) (justify right bottom))
-  )
-  (label "LIDAR_RX" (at 127 101.6 180) (fields_autoplaced)
+  (label "LIDAR_TX" (at 194.31 40.64 180) (fields_autoplaced)
+    (effects (font (size 1.27 1.27)) (justify right bottom))
+  )
+  (label "LIDAR_RX" (at 194.31 43.18 180) (fields_autoplaced)
     (effects (font (size 1.27 1.27)) (justify right bottom))
   )
@@
     (effects (font (size 1.27 1.27)) (justify right bottom))
   )
-  (label "BUMPER2" (at 132.08 86.36 180) (fields_autoplaced)
+  (label "BUMPER2" (at 194.31 101.6 180) (fields_autoplaced)
     (effects (font (size 1.27 1.27)) (justify right bottom))
   )
@@
     (effects (font (size 1.27 1.27)) (justify right bottom))
   )
-  (label "BUMPER3" (at 132.08 88.9 180) (fields_autoplaced)
+  (label "BUMPER3" (at 194.31 99.06 180) (fields_autoplaced)
     (effects (font (size 1.27 1.27)) (justify right bottom))
   )
@@
       (effects (font (size 1.27 1.27)) hide)
     )
-    (pin "4")
     (pin "1")
     (pin "2")
     (pin "3")
+    (pin "4")
     (pin "5")
     (pin "6")

Commit message: routing
Parts:
- added TP101: M1_PWM_FWD, TestPoint:TestPoint_Pad_D1.5mm, symbol Connector:TestPoint
- added TP102: M1_PWM_REV, TestPoint:TestPoint_Pad_D1.5mm, symbol Connector:TestPoint
- added TP103: M2_PWM_FWD, TestPoint:TestPoint_Pad_D1.5mm, symbol Connector:TestPoint
- added TP104: M2_PWM_REV, TestPoint:TestPoint_Pad_D1.5mm, symbol Connector:TestPoint
Connections:
- net BORDER_BACK: now also U101.52 (PD2)
- net BORDER_FRONT: now also U101.53 (PD3)
- net LED_GREEN: now also U101.33 (PB13)
- net LED_ORANGE: now also U101.32 (PB12)
- net LED_RED: now also U101.31 (PB11)
- net LIDAR_DEV_EN: now also U101.26 (PC5)
- net LIDAR_M_EN: now also U101.25 (PC4)
- net M1_PWM_FWD: now also TP101.1
- net M1_PWM_REV: now also TP102.1
- net M2_PWM_FWD: now also TP103.1
- net M2_PWM_REV: now also TP104.1
- net BATT_OUT: now reaches J102.1 (Pin_1), SW101.1 (A)
- net SWO: no longer names the net of J7.8 (Pin_8)
- no-connect marks 6 -> 38
Other:
- moved on the sheet: C101, C102, R101, Y101
